Commit message: update

File: sr_description/urdf/sr_hand.urdf (robot description, URDF)
Before this commit: robot shadowhand_motor, 33 links, 32 joints
Links:
- link rh_ffdistal: geometry collision mesh filename=package://sr_description/meshes/F1.dae scale=0.001 0.001 0.001; visual mesh filename=package://sr_description/meshes/F1.dae scale=0.001 0.001 0.001
- link rh_ffknuckle: geometry collision cylinder length=0.014 radius=0.007; visual mesh filename=package://sr_description/meshes/knuckle.dae scale=0.001 0.001 0.001
- link rh_ffmiddle: geometry collision cylinder length=0.025 radius=0.007; collision sphere radius=0.007
- link rh_ffproximal: geometry collision cylinder length=0.040 radius=0.007; visual mesh filename=package://sr_description/meshes/F3.dae scale=0.001 0.001 0.001
- link rh_forearm: geometry collision box size=0.07 0.07 0.07; collision cylinder length=0.184 radius=0.07
- link rh_lfdistal: geometry collision mesh filename=package://sr_description/meshes/F1.dae scale=0.001 0.001 0.001; visual mesh filename=package://sr_description/meshes/F1.dae scale=0.001 0.001 0.001
- link rh_lfknuckle: geometry collision cylinder length=0.014 radius=0.007; visual mesh filename=package://sr_description/meshes/knuckle.dae scale=0.001 0.001 0.001
- link rh_lfmetacarpal: geometry collision box size=0.018 0.024 0.040; visual mesh filename=package://sr_description/meshes/lfmetacarpal.dae scale=0.001 0.001 0.001
- link rh_lfmiddle: geometry collision cylinder length=0.025 radius=0.007; collision sphere radius=0.007
- link rh_lfproximal: geometry collision cylinder length=0.040 radius=0.007; visual mesh filename=package://sr_description/meshes/F3.dae scale=0.001 0.001 0.001
- link rh_mfdistal: geometry collision mesh filename=package://sr_description/meshes/F1.dae scale=0.001 0.001 0.001; visual mesh filename=package://sr_description/meshes/F1.dae scale=0.001 0.001 0.001
- link rh_mfknuckle: geometry collision cylinder length=0.014 radius=0.007; visual mesh filename=package://sr_description/meshes/knuckle.dae scale=0.001 0.001 0.001
- link rh_mfmiddle: geometry collision cylinder length=0.025 radius=0.007; collision sphere radius=0.007
- link rh_mfproximal: geometry collision cylinder length=0.040 radius=0.007; visual mesh filename=package://sr_description/meshes/F3.dae scale=0.001 0.001 0.001
- link rh_palm: geometry collision box size=0.018 0.024 0.004; collision box size=0.020 0.024 0.040
- link rh_rfdistal: geometry collision mesh filename=package://sr_description/meshes/F1.dae scale=0.001 0.001 0.001; visual mesh filename=package://sr_description/meshes/F1.dae scale=0.001 0.001 0.001
- link rh_rfknuckle: geometry collision cylinder length=0.014 radius=0.007; visual mesh filename=package://sr_description/meshes/knuckle.dae scale=0.001 0.001 0.001
- link rh_rfmiddle: geometry collision cylinder length=0.025 radius=0.007; collision sphere radius=0.007
- link rh_rfproximal: geometry collision cylinder length=0.040 radius=0.007; visual mesh filename=package://sr_description/meshes/F3.dae scale=0.001 0.001 0.001
- link rh_thdistal: geometry collision mesh filename=package://sr_description/meshes/TH1_z.dae scale=0.001 0.001 0.001; visual mesh filename=package://sr_description/meshes/TH1_z.dae scale=0.001 0.001 0.001
- link rh_thmiddle: geometry collision cylinder length=0.018 radius=0.011; collision sphere radius=0.011
- link rh_thproximal: geometry collision cylinder length=0.018 radius=0.012; visual mesh filename=package://sr_description/meshes/TH3_z.dae scale=0.001 0.001 0.001
- link rh_wrist: geometry collision box size=0.027 0.018 0.010; collision box size=0.027 0.018 0.010

File: sr_description/urdf/sr_hand.xacro (robot description, xacro)
@@ -1,8 +1,4 @@
-<?xml version="1.0" ?>
-<!-- =================================================================================== -->
-<!-- |    This document was autogenerated by xacro from file://home/mike/shadow_robot/base/src/sr_common/sr_description/robots/shadowhand_motor.urdf.xacro | -->
-<!-- |    EDITING THIS FILE BY HAND IS NOT RECOMMENDED                                 | -->
-<!-- =================================================================================== -->
-<robot name="shadowhand_motor" xmlns:body="http://playerstage.sourceforge.net/gazebo/xmlschema/#body" xmlns:controller="http://playerstage.sourceforge.net/gazebo/xmlschema/#controller" xmlns:geom="http://playerstage.sourceforge.net/gazebo/xmlschema/#geom" xmlns:interface="http://playerstage.sourceforge.net/gazebo/xmlschema/#interface" xmlns:joint="http://playerstage.sourceforge.net/gazebo/xmlschema/#slider" xmlns:sensor="http://playerstage.sourceforge.net/gazebo/xmlschema/#sensor" xmlns:xacro="http://www.ros.org/wiki/xacro">
+<?xml version="1.0" encoding="utf-8"?>
+<robot name="shadowhand_motor" xmlns:body="http://playerstage.sourceforge.net/gazebo/xmlschema/#body" xmlns:controller="http://playerstage.sourceforge.net/gazebo/xmlschema/#controller" xmlns:geom="http://playerstage.sourceforge.net/gazebo/xmlschema/#geom" xmlns:interface="http://playerstage.sourceforge.net/gazebo/xmlschema/#interface" xmlns:joint="http://playerstage.sourceforge.net/gazebo/xmlschema/#slider" xmlns:sensor="http://playerstage.sourceforge.net/gazebo/xmlschema/#sensor">
   <material name="Blue">
     <color rgba="0.0 0.0 0.8 1.0"/>
@@ -28,4 +24,5 @@
   <gazebo>
     <plugin filename="libgazebo_ros_control.so" name="gazebo_ros_control">
+      <namespace>/shadow_robot</namespace>
     </plugin>
   </gazebo>
@@ -134,9 +131,9 @@
     <actuator name="rh_WRJ2">
       <mechanicalReduction>1</mechanicalReduction>
-      <hardwareInterface>EffortJointInterface</hardwareInterface>
+      <!--<hardwareInterface>EffortJointInterface</hardwareInterface>-->
       <hardwareInterface>PositionJointInterface</hardwareInterface>
     </actuator>
     <joint name="rh_WRJ2">
-      <hardwareInterface>EffortJointInterface</hardwareInterface>
+      <!--<hardwareInterface>EffortJointInterface</hardwareInterface>-->
       <hardwareInterface>PositionJointInterface</hardwareInterface>
     </joint>
@@ -241,9 +238,9 @@
     <actuator name="rh_WRJ1">
       <mechanicalReduction>1</mechanicalReduction>
-      <hardwareInterface>EffortJointInterface</hardwareInterface>
+      <!--<hardwareInterface>EffortJointInterface</hardwareInterface>-->
       <hardwareInterface>PositionJointInterface</hardwareInterface>
     </actuator>
     <joint name="rh_WRJ1">
-      <hardwareInterface>EffortJointInterface</hardwareInterface>
+      <!--<hardwareInterface>EffortJointInterface</hardwareInterface>-->
       <hardwareInterface>PositionJointInterface</hardwareInterface>
     </joint>
@@ -303,9 +300,9 @@
     <actuator name="rh_FFJ4">
       <mechanicalReduction>1</mechanicalReduction>
-      <hardwareInterface>EffortJointInterface</hardwareInterface>
+      <!--<hardwareInterface>EffortJointInterface</hardwareInterface>-->
       <hardwareInterface>PositionJointInterface</hardwareInterface>
     </actuator>
     <joint name="rh_FFJ4">
-      <hardwareInterface>EffortJointInterface</hardwareInterface>
+      <!--<hardwareInterface>EffortJointInterface</hardwareInterface>-->
       <hardwareInterface>PositionJointInterface</hardwareInterface>
     </joint>
@@ -365,9 +362,9 @@
     <actuator name="rh_FFJ3">
       <mechanicalReduction>1</mechanicalReduction>
-      <hardwareInterface>EffortJointInterface</hardwareInterface>
+      <!--<hardwareInterface>EffortJointInterface</hardwareInterface>-->
       <hardwareInterface>PositionJointInterface</hardwareInterface>
     </actuator>
     <joint name="rh_FFJ3">
-      <hardwareInterface>EffortJointInterface</hardwareInterface>
+      <!--<hardwareInterface>EffortJointInterface</hardwareInterface>-->
       <hardwareInterface>PositionJointInterface</hardwareInterface>
     </joint>
@@ -439,9 +436,9 @@
     <actuator name="rh_FFJ2">
       <mechanicalReduction>1</mechanicalReduction>
-      <hardwareInterface>EffortJointInterface</hardwareInterface>
+      <!--<hardwareInterface>EffortJointInterface</hardwareInterface>-->
       <hardwareInterface>PositionJointInterface</hardwareInterface>
     </actuator>
     <joint name="rh_FFJ2">
-      <hardwareInterface>EffortJointInterface</hardwareInterface>
+      <!--<hardwareInterface>EffortJointInterface</hardwareInterface>-->
       <hardwareInterface>PositionJointInterface</hardwareInterface>
     </joint>
@@ -451,9 +448,9 @@
     <actuator name="rh_FFJ1">
       <mechanicalReduction>1</mechanicalReduction>
-      <hardwareInterface>EffortJointInterface</hardwareInterface>
+      <!--<hardwareInterface>EffortJointInterface</hardwareInterface>-->
       <hardwareInterface>PositionJointInterface</hardwareInterface>
     </actuator>
     <joint name="rh_FFJ1">
-      <hardwareInterface>EffortJointInterface</hardwareInterface>
+      <!--<hardwareInterface>EffortJointInterface</hardwareInterface>-->
       <hardwareInterface>PositionJointInterface</hardwareInterface>
     </joint>
@@ -583,9 +580,9 @@
     <actuator name="rh_MFJ4">
       <mechanicalReduction>1</mechanicalReduction>
-      <hardwareInterface>EffortJointInterface</hardwareInterface>
+      <!--<hardwareInterface>EffortJointInterface</hardwareInterface>-->
       <hardwareInterface>PositionJointInterface</hardwareInterface>
     </actuator>
     <joint name="rh_MFJ4">
-      <hardwareInterface>EffortJointInterface</hardwareInterface>
+      <!--<hardwareInterface>EffortJointInterface</hardwareInterface>-->
       <hardwareInterface>PositionJointInterface</hardwareInterface>
     </joint>
@@ -645,9 +642,9 @@
     <actuator name="rh_MFJ3">
       <mechanicalReduction>1</mechanicalReduction>
-      <hardwareInterface>EffortJointInterface</hardwareInterface>
+      <!--<hardwareInterface>EffortJointInterface</hardwareInterface>-->
       <hardwareInterface>PositionJointInterface</hardwareInterface>
     </actuator>
     <joint name="rh_MFJ3">
-      <hardwareInterface>EffortJointInterface</hardwareInterface>
+      <!--<hardwareInterface>EffortJointInterface</hardwareInterface>-->
       <hardwareInterface>PositionJointInterface</hardwareInterface>
     </joint>
@@ -719,9 +716,9 @@
     <actuator name="rh_MFJ2">
       <mechanicalReduction>1</mechanicalReduction>
-      <hardwareInterface>EffortJointInterface</hardwareInterface>
+      <!--<hardwareInterface>EffortJointInterface</hardwareInterface>-->
       <hardwareInterface>PositionJointInterface</hardwareInterface>
     </actuator>
     <joint name="rh_MFJ2">
-      <hardwareInterface>EffortJointInterface</hardwareInterface>
+      <!--<hardwareInterface>EffortJointInterface</hardwareInterface>-->
       <hardwareInterface>PositionJointInterface</hardwareInterface>
     </joint>
@@ -731,9 +728,9 @@
     <actuator name="rh_MFJ1">
       <mechanicalReduction>1</mechanicalReduction>
-      <hardwareInterface>EffortJointInterface</hardwareInterface>
+      <!--<hardwareInterface>EffortJointInterface</hardwareInterface>-->
       <hardwareInterface>PositionJointInterface</hardwareInterface>
     </actuator>
     <joint name="rh_MFJ1">
-      <hardwareInterface>EffortJointInterface</hardwareInterface>
+      <!--<hardwareInterface>EffortJointInterface</hardwareInterface>-->
       <hardwareInterface>PositionJointInterface</hardwareInterface>
     </joint>
@@ -863,9 +860,9 @@
     <actuator name="rh_RFJ4">
       <mechanicalReduction>1</mechanicalReduction>
-      <hardwareInterface>EffortJointInterface</hardwareInterface>
+      <!--<hardwareInterface>EffortJointInterface</hardwareInterface>-->
       <hardwareInterface>PositionJointInterface</hardwareInterface>
     </actuator>
     <joint name="rh_RFJ4">
-      <hardwareInterface>EffortJointInterface</hardwareInterface>
+      <!--<hardwareInterface>EffortJointInterface</hardwareInterface>-->
       <hardwareInterface>PositionJointInterface</hardwareInterface>
     </joint>
@@ -925,9 +922,9 @@
     <actuator name="rh_RFJ3">
       <mechanicalReduction>1</mechanicalReduction>
-      <hardwareInterface>EffortJointInterface</hardwareInterface>
+      <!--<hardwareInterface>EffortJointInterface</hardwareInterface>-->
       <hardwareInterface>PositionJointInterface</hardwareInterface>
     </actuator>
     <joint name="rh_RFJ3">
-      <hardwareInterface>EffortJointInterface</hardwareInterface>
+      <!--<hardwareInterface>EffortJointInterface</hardwareInterface>-->
       <hardwareInterface>PositionJointInterface</hardwareInterface>
     </joint>
@@ -999,9 +996,9 @@
     <actuator name="rh_RFJ2">
       <mechanicalReduction>1</mechanicalReduction>
-      <hardwareInterface>EffortJointInterface</hardwareInterface>
+      <!--<hardwareInterface>EffortJointInterface</hardwareInterface>-->
       <hardwareInterface>PositionJointInterface</hardwareInterface>
     </actuator>
     <joint name="rh_RFJ2">
-      <hardwareInterface>EffortJointInterface</hardwareInterface>
+      <!--<hardwareInterface>EffortJointInterface</hardwareInterface>-->
       <hardwareInterface>PositionJointInterface</hardwareInterface>
     </joint>
@@ -1011,9 +1008,9 @@
     <actuator name="rh_RFJ1">
       <mechanicalReduction>1</mechanicalReduction>
-      <hardwareInterface>EffortJointInterface</hardwareInterface>
+      <!--<hardwareInterface>EffortJointInterface</hardwareInterface>-->
       <hardwareInterface>PositionJointInterface</hardwareInterface>
     </actuator>
     <joint name="rh_RFJ1">
-      <hardwareInterface>EffortJointInterface</hardwareInterface>
+      <!--<hardwareInterface>EffortJointInterface</hardwareInterface>-->
       <hardwareInterface>PositionJointInterface</hardwareInterface>
     </joint>
@@ -1142,9 +1139,9 @@
     <actuator name="rh_LFJ5">
       <mechanicalReduction>1</mechanicalReduction>
-      <hardwareInterface>EffortJointInterface</hardwareInterface>
+      <!--<hardwareInterface>EffortJointInterface</hardwareInterface>-->
       <hardwareInterface>PositionJointInterface</hardwareInterface>
     </actuator>
     <joint name="rh_LFJ5">
-      <hardwareInterface>EffortJointInterface</hardwareInterface>
+      <!--<hardwareInterface>EffortJointInterface</hardwareInterface>-->
       <hardwareInterface>PositionJointInterface</hardwareInterface>
     </joint>
@@ -1205,9 +1202,9 @@
     <actuator name="rh_LFJ4">
       <mechanicalReduction>1</mechanicalReduction>
-      <hardwareInterface>EffortJointInterface</hardwareInterface>
+      <!--<hardwareInterface>EffortJointInterface</hardwareInterface>-->
       <hardwareInterface>PositionJointInterface</hardwareInterface>
     </actuator>
     <joint name="rh_LFJ4">
-      <hardwareInterface>EffortJointInterface</hardwareInterface>
+      <!--<hardwareInterface>EffortJointInterface</hardwareInterface>-->
       <hardwareInterface>PositionJointInterface</hardwareInterface>
     </joint>
@@ -1267,9 +1264,9 @@
     <actuator name="rh_LFJ3">
       <mechanicalReduction>1</mechanicalReduction>
-      <hardwareInterface>EffortJointInterface</hardwareInterface>
+      <!--<hardwareInterface>EffortJointInterface</hardwareInterface>-->
       <hardwareInterface>PositionJointInterface</hardwareInterface>
     </actuator>
     <joint name="rh_LFJ3">
-      <hardwareInterface>EffortJointInterface</hardwareInterface>
+      <!--<hardwareInterface>EffortJointInterface</hardwareInterface>-->
       <hardwareInterface>PositionJointInterface</hardwareInterface>
     </joint>
@@ -1341,9 +1338,9 @@
     <actuator name="rh_LFJ2">
       <mechanicalReduction>1</mechanicalReduction>
-      <hardwareInterface>EffortJointInterface</hardwareInterface>
+      <!--<hardwareInterface>EffortJointInterface</hardwareInterface>-->
       <hardwareInterface>PositionJointInterface</hardwareInterface>
     </actuator>
     <joint name="rh_LFJ2">
-      <hardwareInterface>EffortJointInterface</hardwareInterface>
+      <!--<hardwareInterface>EffortJointInterface</hardwareInterface>-->
       <hardwareInterface>PositionJointInterface</hardwareInterface>
     </joint>
@@ -1353,9 +1350,9 @@
     <actuator name="rh_LFJ1">
       <mechanicalReduction>1</mechanicalReduction>
-      <hardwareInterface>EffortJointInterface</hardwareInterface>
+      <!--<hardwareInterface>EffortJointInterface</hardwareInterface>-->
       <hardwareInterface>PositionJointInterface</hardwareInterface>
     </actuator>
     <joint name="rh_LFJ1">
-      <hardwareInterface>EffortJointInterface</hardwareInterface>
+      <!--<hardwareInterface>EffortJointInterface</hardwareInterface>-->
       <hardwareInterface>PositionJointInterface</hardwareInterface>
     </joint>
@@ -1486,9 +1483,9 @@
     <actuator name="rh_THJ5">
       <mechanicalReduction>1</mechanicalReduction>
-      <hardwareInterface>EffortJointInterface</hardwareInterface>
+      <!--<hardwareInterface>EffortJointInterface</hardwareInterface>-->
       <hardwareInterface>PositionJointInterface</hardwareInterface>
     </actuator>
     <joint name="rh_THJ5">
-      <hardwareInterface>EffortJointInterface</hardwareInterface>
+      <!--<hardwareInterface>EffortJointInterface</hardwareInterface>-->
       <hardwareInterface>PositionJointInterface</hardwareInterface>
     </joint>
@@ -1550,9 +1547,9 @@
     <actuator name="rh_THJ4">
       <mechanicalReduction>1</mechanicalReduction>
-      <hardwareInterface>EffortJointInterface</hardwareInterface>
+      <!--<hardwareInterface>EffortJointInterface</hardwareInterface>-->
       <hardwareInterface>PositionJointInterface</hardwareInterface>
     </actuator>
     <joint name="rh_THJ4">
-      <hardwareInterface>EffortJointInterface</hardwareInterface>
+      <!--<hardwareInterface>EffortJointInterface</hardwareInterface>-->
       <hardwareInterface>PositionJointInterface</hardwareInterface>
     </joint>
@@ -1614,9 +1611,9 @@
     <actuator name="rh_THJ3">
       <mechanicalReduction>1</mechanicalReduction>
-      <hardwareInterface>EffortJointInterface</hardwareInterface>
+      <!--<hardwareInterface>EffortJointInterface</hardwareInterface>-->
       <hardwareInterface>PositionJointInterface</hardwareInterface>
     </actuator>
     <joint name="rh_THJ3">
-      <hardwareInterface>EffortJointInterface</hardwareInterface>
+      <!--<hardwareInterface>EffortJointInterface</hardwareInterface>-->
       <hardwareInterface>PositionJointInterface</hardwareInterface>
     </joint>
@@ -1684,9 +1681,9 @@
     <actuator name="rh_THJ2">
       <mechanicalReduction>1</mechanicalReduction>
-      <hardwareInterface>EffortJointInterface</hardwareInterface>
+      <!--<hardwareInterface>EffortJointInterface</hardwareInterface>-->
       <hardwareInterface>PositionJointInterface</hardwareInterface>
     </actuator>
     <joint name="rh_THJ2">
-      <hardwareInterface>EffortJointInterface</hardwareInterface>
+      <!--<hardwareInterface>EffortJointInterface</hardwareInterface>-->
       <hardwareInterface>PositionJointInterface</hardwareInterface>
     </joint>
@@ -1785,9 +1782,9 @@
     <actuator name="rh_THJ1">
       <mechanicalReduction>1</mechanicalReduction>
-      <hardwareInterface>EffortJointInterface</hardwareInterface>
+      <!--<hardwareInterface>EffortJointInterface</hardwareInterface>-->
       <hardwareInterface>PositionJointInterface</hardwareInterface>
     </actuator>
     <joint name="rh_THJ1">
-      <hardwareInterface>EffortJointInterface</hardwareInterface>
+      <!--<hardwareInterface>EffortJointInterface</hardwareInterface>-->
       <hardwareInterface>PositionJointInterface</hardwareInterface>
     </joint>
